File: Kicad/_saved_GrowChamberSensorPuck.sch (KiCad schematic (older format))
At the start: 13 parts, among them P1 CONN_01X07, U1 Si7006, U2 CCS811

Commit message: added footprints to sensor puck
Parts:
- P1: footprint (none) -> TheLeafSpa:7 POS Arduino Header
- R8: footprint (none) -> Resistors_SMD:R_0805
- U2: footprint (none) -> TheLeafSpa:CCS811
Changed lines of the file:
@@
 F 0 "U2" H 6550 2600 60  0000 C CNN
 F 1 "CCS811" H 6900 2600 60  0000 C CNN
-F 2 "" H 6900 1850 60  0001 C CNN
+F 2 "TheLeafSpa:CCS811" H 6900 1850 60  0001 C CNN
 F 3 "" H 6900 1850 60  0001 C CNN
 F 4 "CCS811CT-ND" H 6900 1850 60  0001 C CNN "PN"
@@
 F 0 "R8" V 8780 1800 50  0000 C CNN
 F 1 "NTC100KΩ" V 8700 1800 50  0000 C CNN
-F 2 "" V 8630 1800 50  0001 C CNN
+F 2 "Resistors_SMD:R_0805" V 8630 1800 50  0001 C CNN
 F 3 "" H 8700 1800 50  0000 C CNN
 F 4 "NTCS0805E3104FXT" H 8700 1800 60  0001 C CNN "PN"
@@
 F 0 "P1" H 1800 2400 50  0000 C CNN
 F 1 "CONN_01X07" V 1900 2000 50  0000 C CNN
-F 2 "" H 1800 2000 50  0001 C CNN
+F 2 "TheLeafSpa:7 POS Arduino Header" H 1800 2000 50  0001 C CNN
 F 3 "" H 1800 2000 50  0000 C CNN
 	1    1800 2000

Commit message: Feb 15 update
Parts:
- U1: footprint (none) -> TheLeafSpa:Si7006
Changed lines of the file:
@@
 F 0 "U1" H 3400 5100 60  0000 C CNN
 F 1 "Si7006" H 3350 6100 60  0000 C CNN
-F 2 "" H 3750 5500 60  0001 C CNN
+F 2 "TheLeafSpa:Si7006" H 3750 5500 60  0001 C CNN
 F 3 "" H 3750 5500 60  0001 C CNN
 F 4 "SI7006-A20-IM" H 3750 5500 60  0001 C CNN "PN"
