File: Kicad/_saved_GrowChamberSensorPuck.sch (KiCad schematic (older format))
At the start: 13 parts, among them P1 CONN_01X07, U1 Si7006, U2 CCS811

Commit message: updated TheLeafSpa.ino after first tests
Parts:
- JP1: footprint Socket_Strips:Socket_Strip_Straight_1x02_Pitch2.54mm -> TheLeafSpa:Jumper_2_Pad
Connections:
- net SCL: now also P1.5 (P5); no longer P1.4 (P4)
- net SDA: now also P1.4 (P4); no longer P1.5 (P5)
- net +3.3v: no longer names the net of C2.2, U2.6 (VDD)
Changed lines of the file:
@@
 F 0 "JP1" H 4950 2530 50  0000 C CNN
 F 1 "JMPR" H 4960 2390 50  0000 C CNN
-F 2 "Socket_Strips:Socket_Strip_Straight_1x02_Pitch2.54mm" H 4950 2450 50  0001 C CNN
+F 2 "TheLeafSpa:Jumper_2_Pad" H 4950 2450 50  0001 C CNN
 F 3 "" H 4950 2450 50  0000 C CNN
 F 4 "X" H 4950 2450 60  0001 C CNN "PN"
@@
 NRESET
 Text GLabel 9400 2600 0    60   Input ~ 0
-SCL
+SDA
 Text GLabel 9400 2700 0    60   Input ~ 0
-SDA
+SCL
 $Comp
 L GNDD #PWR010
@@
 	9450 2500 9450 3300
 Connection ~ 9450 2500
-Text Label 3500 1350 0    60   ~ 0
-+3.3v
 $EndSCHEMATC
