File: Kicad/GrowChamberSensorPuck.sch (KiCad schematic (older format))
At the start: 13 parts, among them P1 CONN_01X07, U1 Si7006, U2 CCS811

Commit message: evolved Grow Sensor Puck schematic
Parts:
- removed P1: CONN_01X07, symbol CONN_01X07
- removed R6: 4K7, Capacitors_SMD:C_0805_HandSoldering, symbol R
- removed R8: NTC100KΩ, symbol R
- added JP1: Jumper_NO_Small, symbol Jumper_NO_Small
- added P1: CONN_01X04, symbol CONN_01X04
- added P2: CONN_01X03, symbol CONN_01X03
- added TH1: OPT, symbol Thermistor
- C2: value 4.7uF -> 4.7u
- R1, R2, R3: value 10K -> 4.7K
- R4: value 10K -> 100K
- R5: value 4K7 -> 100K
- R7: value 100K -> 10K
- U1: footprint (none) -> TheLeafSpa:Si7006
- U2: footprint (none) -> TheLeafSpa:CCS811
Connections:
- net labels added: +3.3V, NTC_SENSE
- net labels removed: PWM, SENSE, VDD
- wire segments 45 -> 48
Other:
- note added: "I2C ADDR\nOpen (Default) - 0x5B\nClosed - 0x5A"
- moved on the sheet: C1, C2, R1, R5, R7, U2

Commit message: updated GrowChamberSensorPuck Kicad stuff
Parts:
- removed P1: CONN_01X04, symbol CONN_01X04
- removed P2: CONN_01X03, symbol CONN_01X03
- removed TH1: OPT, symbol Thermistor
- added P1: CONN_01X07, Socket_Strips:Socket_Strip_Straight_1x07_Pitch2.54mm, symbol CONN_01X07
- added TH1: Thermistor_NTC, Socket_Strips:Socket_Strip_Straight_1x02_Pitch2.54mm, symbol Thermistor_NTC
- C2: value 4.7u -> 1u
- JP1: value Jumper_NO_Small -> JMPR; footprint (none) -> Socket_Strips:Socket_Strip_Straight_1x02_Pitch2.54mm
- R1, R2, R3: value 4.7K -> 4K7
Connections:
- net +3V3: now also P1.6 (P6)
- net AUX: now also TH1.1
- net GNDD: now also P1.7 (P7)
- net NINT: now also P1.2 (P2)
- net NRESET: now also P1.1 (P1)
- net NTC_SENSE: now also TH1.2
- net NWAKE: now also P1.3 (P3)
- net SCL: now also P1.4 (P4)
- net SDA: now also P1.5 (P5)
- net +3.3v: now reaches C2.2, U2.6 (VDD)
Other:
- moved on the sheet: R4

Commit message: updated TheLeafSpa.ino after first tests
Connections:
- net SCL: now also P1.5 (P5); no longer P1.4 (P4)
- net SDA: now also P1.4 (P4); no longer P1.5 (P5)
Changed lines of the file:
@@
 NRESET
 Text GLabel 9400 2600 0    60   Input ~ 0
+SDA
+Text GLabel 9400 2700 0    60   Input ~ 0
 SCL
-Text GLabel 9400 2700 0    60   Input ~ 0
-SDA
 $Comp
 L GNDD #PWR010

Commit message: cleaned up files
Parts:
- JP1: footprint Socket_Strips:Socket_Strip_Straight_1x02_Pitch2.54mm -> TheLeafSpa:Jumper_2_Pad
Connections:
- net +3.3v: no longer names the net of C2.2, U2.6 (VDD)
Changed lines of the file:
@@
 F 0 "JP1" H 4950 2530 50  0000 C CNN
 F 1 "JMPR" H 4960 2390 50  0000 C CNN
-F 2 "Socket_Strips:Socket_Strip_Straight_1x02_Pitch2.54mm" H 4950 2450 50  0001 C CNN
+F 2 "TheLeafSpa:Jumper_2_Pad" H 4950 2450 50  0001 C CNN
 F 3 "" H 4950 2450 50  0000 C CNN
 F 4 "X" H 4950 2450 60  0001 C CNN "PN"
@@
 	9450 2500 9450 3300
 Connection ~ 9450 2500
-Text Label 3500 1350 0    60   ~ 0
-+3.3v
 $EndSCHEMATC
